File: ring.kicad_pcb (KiCad board)
At the start: 2 copper layers, 38 x 10 mm, 30 parts, among them J1 5034800240, J2 5034800440, Q1 IRLML6344TRPBF, U1 ANNA-B112-02B, U2 LSM6DSV16X

Commit message: Sync board after router C-A* port and hole-to-hole fix
The monorepo router now runs its via-penalty and corridor costs in the
C accelerator; re-routing under C tie-breaking removed all three
negative-annular via-in-pads on U2, cut total trace 576 -> 502 mm
(83 -> 81 vias), and a new net-independent drill-spacing guard
relocated one GND stitch via. Verified on this repo's pair:
kicad-cli DRC + schematic parity 0 errors / 0 warnings / 0 unconnected.
Gerber + drill set and the top/bottom preview regenerated;
preview-3d (the fold illustration, geometry unchanged) kept as-is.

Co-Authored-By: Claude Fable 5 <noreply@anthropic.com>
Routing:
- net LED_GREEN: track 65.1 -> 44.9 mm, vias 8 -> 6
- net VBUS: track 40.7 -> 21.5 mm, vias 0 -> 2
- net VBAT: track 84.4 -> 66.1 mm, vias 17 -> 10
- net SDA: track 30.3 -> 23.0 mm, vias 5 -> 2
- net QVAR1_RAW: track 6.25 -> 12.5 mm, vias 0 -> 2
- net QVAR2: track 20.2 -> 14.2 mm, vias 5 -> 0
- net QVAR1: track 21.0 -> 15.4 mm, vias 2 -> 6
- net SWDIO: track 20.6 -> 15.8 mm, vias 2 -> 6
- net LED_GREEN_A: track 19.7 -> 15.4 mm, vias 2 -> 4
- net SWDCLK: track 9.95 -> 13.8 mm
- net SCL: track 23.9 -> 21.2 mm, vias 3 -> 6
- net MOTOR_N: track 14.7 -> 16.9 mm, vias 4 -> 3
- net HAPTIC_EN: track 31.9 -> 34.1 mm, vias 6 -> 2
- net LED_RED_A: track 16.3 -> 14.4 mm, vias 2 -> 4
- net QVAR2_RAW: track 6.26 -> 4.54 mm
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
Commit message: Sync board after via-in-pad guard hardening
The monorepo router now enforces a commit-time annular floor for
terminating vias (rejects below-floor via-in-pad before commit, loud
actionable failures) and re-routed the ring under it. This board keeps
its 23 adequate-annular via-in-pads (all >= +0.075 mm ring; the
poking-past class is extinct) with zero negative-annular and zero
hole-to-hole findings. Verified on this repo's pair: kicad-cli DRC +
schematic parity 0 errors / 0 warnings / 0 unconnected. Gerber + drill
set and top/bottom preview regenerated.

Co-Authored-By: Claude Fable 5 <noreply@anthropic.com>
Routing:
- net GND: track 111.9 -> 103.3 mm, vias 16 -> 15
- net QVAR1_RAW: track 12.5 -> 6.91 mm
- net VBAT: track 66.1 -> 61.5 mm
- net HAPTIC_EN: track 34.1 -> 32.6 mm, vias 2 -> 0
- net QVAR2: track 14.2 -> 15.1 mm
